File: Portable Offline Translator/IO.kicad_sch (KiCad schematic)
At the start: 5 parts

Commit message: Added Datasheets and PCB
Parts:
- removed LS?: Speaker, symbol Device:Speaker
- added J201: Conn_01x10_Female, Connector_PinSocket_2.54mm:PinSocket_1x10_P2.54mm_Vertical, symbol Connector:Conn_01x10_Female
- added LS201: CMS-16098A-SP, CMS_16098A_SP(Speaker):CUI_CMS-16098A-SP, symbol CMS-16098A-SP:CMS-16098A-SP
- MK201: renamed from MK?; footprint ICS-43434:MIC_ICS-43434 -> ICS_43434(MIC):MIC_ICS-43434
- R201, R202: renamed from R?; footprint (none) -> Resistor_SMD:R_0805_2012Metric_Pad1.20x1.40mm_HandSolder
- U201: renamed from U?; footprint 21-0896B_9_MXM -> MAX98357AEWL_T(Audio Amp):21-0896B_9_MXM
Connections:
- net OUTN: now also LS201.N
- net OUTP: now also LS201.P
- new net I2C1_SCL: J201.1 (Pin_1)
- new net I2C1_SDA: J201.2 (Pin_2)
- new net LCD_Data/Command: J201.3 (Pin_3)
- new net LCD_GND: J201.9 (Pin_9)
- new net LCD_RST: J201.4 (Pin_4)
- new net LCD_VIN: J201.10 (Pin_10)
- new net SPI1_MOSI: J201.6 (Pin_6)
- new net SPI1_NSS: J201.5 (Pin_5)
- new net SPI1_SCK: J201.8 (Pin_8)
- new net SPI_MISO: J201.7 (Pin_7)
Other:
- note added: "LCD and PI Connection"
- note removed: "LCD"

Commit message: PCB Backup
Parts:
- removed J201: Conn_01x10_Female, Connector_PinSocket_2.54mm:PinSocket_1x10_P2.54mm_Vertical, symbol Connector:Conn_01x10_Female
- added J201: Conn_01x08_Male, Connector_PinSocket_2.54mm:PinSocket_1x08_P2.54mm_Vertical, symbol Connector:Conn_01x08_Male
Connections:
- net LCD_Data/Command: now also J201.7 (Pin_7)
- net LCD_GND: now also J201.2 (Pin_2)
- net LCD_RST: now also J201.8 (Pin_8)
- net SPI1_MOSI: now also J201.5 (Pin_5)
- net SPI1_NSS: now also J201.6 (Pin_6)
- net SPI1_SCK: now also J201.4 (Pin_4)
- net SPI_MISO: now also J201.3 (Pin_3)
- new net LCD_VCC: J201.1 (Pin_1)
Changed lines of the file:
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@@
+    (stroke (width 0) (type default) (color 0 0 0 0))
+  )
+  (wire (pts (xy 171.45 109.22) (xy 165.1 109.22))
     (stroke (width 0) (type default) (color 0 0 0 0))
   )
@@
     (stroke (width 0) (type default) (color 0 0 0 0))
   )
-  (wire (pts (xy 233.68 129.54) (xy 227.33 129.54))
-    (stroke (width 0) (type default) (color 0 0 0 0))
-  )
   (wire (pts (xy 149.86 62.23) (xy 152.4 62.23))
     (stroke (width 0) (type default) (color 0 0 0 0))
   )
-  (wire (pts (xy 233.68 132.08) (xy 227.33 132.08))
+  (wire (pts (xy 171.45 119.38) (xy 165.1 119.38))
     (stroke (width 0) (type default) (color 0 0 0 0))
   )
@@
     (stroke (width 0) (type default) (color 0 0 0 0))
   )
-  (wire (pts (xy 233.68 127) (xy 227.33 127))
-    (stroke (width 0) (type default) (color 0 0 0 0))
-  )
   (wire (pts (xy 73.66 44.45) (xy 73.66 46.99))
     (stroke (width 0) (type default) (color 0 0 0 0))
   )
-  (wire (pts (xy 233.68 114.3) (xy 227.33 114.3))
-    (stroke (width 0) (type default) (color 0 0 0 0))
-  )
-  (wire (pts (xy 233.68 116.84) (xy 227.33 116.84))
-    (stroke (width 0) (type default) (color 0 0 0 0))
-  )
-  (wire (pts (xy 233.68 109.22) (xy 227.33 109.22))
-    (stroke (width 0) (type default) (color 0 0 0 0))
-  )
   (wire (pts (xy 119.38 130.81) (xy 119.38 144.78))
     (stroke (width 0) (type default) (color 0 0 0 0))
@@
     (stroke (width 0) (type default) (color 0 0 0 0))
   )
+  (wire (pts (xy 171.45 116.84) (xy 165.1 116.84))
+    (stroke (width 0) (type default) (color 0 0 0 0))
+  )
   (wire (pts (xy 40.64 130.81) (xy 40.64 128.27))
     (stroke (width 0) (type default) (color 0 0 0 0))
   )
+  (wire (pts (xy 171.45 114.3) (xy 165.1 114.3))
+    (stroke (width 0) (type default) (color 0 0 0 0))
+  )
   (wire (pts (xy 184.15 67.31) (xy 184.15 73.66))
     (stroke (width 0) (type default) (color 0 0 0 0))
   )
+  (wire (pts (xy 171.45 121.92) (xy 165.1 121.92))
+    (stroke (width 0) (type default) (color 0 0 0 0))
+  )
   (wire (pts (xy 179.07 46.99) (xy 184.15 46.99))
     (stroke (width 0) (type default) (color 0 0 0 0))
   )
-  (wire (pts (xy 233.68 121.92) (xy 227.33 121.92))
-    (stroke (width 0) (type default) (color 0 0 0 0))
-  )
-  (wire (pts (xy 233.68 124.46) (xy 227.33 124.46))
+  (wire (pts (xy 171.45 111.76) (xy 165.1 111.76))
     (stroke (width 0) (type default) (color 0 0 0 0))
   )
@@
     (stroke (width 0) (type default) (color 0 0 0 0))
   )
-  (wire (pts (xy 233.68 119.38) (xy 227.33 119.38))
-    (stroke (width 0) (type default) (color 0 0 0 0))
-  )
   (wire (pts (xy 73.66 59.69) (xy 73.66 57.15))
     (stroke (width 0) (type default) (color 0 0 0 0))
   )
+  (wire (pts (xy 171.45 104.14) (xy 165.1 104.14))
+    (stroke (width 0) (type default) (color 0 0 0 0))
+  )
   (wire (pts (xy 46.99 130.81) (xy 40.64 130.81))
     (stroke (width 0) (type default) (color 0 0 0 0))
   )
-  (wire (pts (xy 233.68 111.76) (xy 227.33 111.76))
+  (wire (pts (xy 171.45 106.68) (xy 165.1 106.68))
     (stroke (width 0) (type default) (color 0 0 0 0))
   )
@@
     (effects (font (size 3 3) (thickness 0.6) bold) (justify left bottom))
   )
-  (text "LCD and PI Connection\n" (at 208.28 101.6 0)
+  (text "LCD and PI Connection\n" (at 214.63 17.78 0)
     (effects (font (size 3 3) (thickness 0.6) bold) (justify left bottom))
   )
@@
     (effects (font (size 1.27 1.27)) (justify right bottom))
   )
-  (hierarchical_label "LCD_Data{slash}Command" (shape input) (at 233.68 127 0)
-    (effects (font (size 1.27 1.27)) (justify left))
-  )
-  (hierarchical_label "LCD_RST" (shape input) (at 233.68 124.46 0)
+  (hierarchical_label "LCD_GND" (shape input) (at 171.45 106.68 0)
+    (effects (font (size 1.27 1.27)) (justify left))
+  )
+  (hierarchical_label "SPI_MISO" (shape output) (at 171.45 109.22 0)
     (effects (font (size 1.27 1.27)) (justify left))
   )
@@
     (effects (font (size 1.27 1.27)) (justify right))
   )
-  (hierarchical_label "SPI_MISO" (shape output) (at 233.68 116.84 0)
-    (effects (font (size 1.27 1.27)) (justify left))
-  )
-  (hierarchical_label "I2C1_SDA" (shape bidirectional) (at 233.68 129.54 0)
+  (hierarchical_label "SPI1_NSS" (shape input) (at 171.45 116.84 0)
+    (effects (font (size 1.27 1.27)) (justify left))
+  )
+  (hierarchical_label "LCD_Data{slash}Command" (shape input) (at 171.45 119.38 0)
+    (effects (font (size 1.27 1.27)) (justify left))
+  )
+  (hierarchical_label "SPI1_SCK" (shape input) (at 171.45 111.76 0)
     (effects (font (size 1.27 1.27)) (justify left))
   )
@@
     (effects (font (size 1.27 1.27)) (justify right))
   )
+  (hierarchical_label "LCD_RST" (shape input) (at 171.45 121.92 0)
+    (effects (font (size 1.27 1.27)) (justify left))
+  )
   (hierarchical_label "MIC_I2S3_SD" (shape output) (at 149.86 62.23 180)
     (effects (font (size 1.27 1.27)) (justify right))
   )
-  (hierarchical_label "LCD_VIN" (shape input) (at 233.68 109.22 0)
+  (hierarchical_label "LCD_VCC" (shape input) (at 171.45 104.14 0)
     (effects (font (size 1.27 1.27)) (justify left))
   )
@@
     (effects (font (size 1.27 1.27)) (justify left))
   )
-  (hierarchical_label "I2C1_SCL" (shape input) (at 233.68 132.08 0)
-    (effects (font (size 1.27 1.27)) (justify left))
-  )
-  (hierarchical_label "LCD_GND" (shape input) (at 233.68 111.76 0)
-    (effects (font (size 1.27 1.27)) (justify left))
-  )
-  (hierarchical_label "SPI1_SCK" (shape input) (at 233.68 114.3 0)
+  (hierarchical_label "SPI1_MOSI" (shape input) (at 171.45 114.3 0)
     (effects (font (size 1.27 1.27)) (justify left))
   )
   (hierarchical_label "AMP_I2S2_CK" (shape input) (at 107.95 133.35 0)
-    (effects (font (size 1.27 1.27)) (justify left))
-  )
-  (hierarchical_label "SPI1_MOSI" (shape input) (at 233.68 119.38 0)
-    (effects (font (size 1.27 1.27)) (justify left))
-  )
-  (hierarchical_label "SPI1_NSS" (shape input) (at 233.68 121.92 0)
     (effects (font (size 1.27 1.27)) (justify left))
   )
@@
     )
     (pin "1")
-  )
-  (symbol (lib_id "Connector:Conn_01x10_Female") (at 222.25 121.92 180) (unit 1)
-    (in_bom yes) (on_board yes) (fields_autoplaced)
-    (property "Reference" "J201" (id 0) (at 222.885 104.14 0))
-    (property "Value" "Conn_01x10_Female" (id 1) (at 222.885 106.68 0))
-    (property "Footprint" "Connector_PinSocket_2.54mm:PinSocket_1x10_P2.54mm_Vertical" (id 2) (at 222.25 121.92 0)
-      (effects (font (size 1.27 1.27)) hide)
-    )
-    (property "Datasheet" "~" (id 3) (at 222.25 121.92 0)
-      (effects (font (size 1.27 1.27)) hide)
-    )
-    (pin "1")
-    (pin "10")
-    (pin "2")
-    (pin "3")
-    (pin "4")
-    (pin "5")
-    (pin "6")
-    (pin "7")
-    (pin "8")
-    (pin "9")
   )
   (symbol (lib_id "2025-02-27_21-45-42:MAX98357AEWL+T") (at 46.99 128.27 0) (unit 1)
@@
     (pin "P")
   )
+  (symbol (lib_id "Connector:Conn_01x08_Male") (at 160.02 111.76 0) (unit 1)
+    (in_bom yes) (on_board yes) (fields_autoplaced)
+    (property "Reference" "J201" (id 0) (at 160.655 99.06 0))
+    (property "Value" "Conn_01x08_Male" (id 1) (at 160.655 101.6 0))
+    (property "Footprint" "Connector_PinSocket_2.54mm:PinSocket_1x08_P2.54mm_Vertical" (id 2) (at 160.02 111.76 0)
+      (effects (font (size 1.27 1.27)) hide)
+    )
+    (property "Datasheet" "~" (id 3) (at 160.02 111.76 0)
+      (effects (font (size 1.27 1.27)) hide)
+    )
+    (pin "1")
+    (pin "2")
+    (pin "3")
+    (pin "4")
+    (pin "5")
+    (pin "6")
+    (pin "7")
+    (pin "8")
+  )
   (symbol (lib_id "power:GND") (at 119.38 147.32 0) (unit 1)
