File: Portable Offline Translator/IO.kicad_sch (KiCad schematic)
At the start: 13 parts, among them J201 Conn_01x08_Male, U202 MAX98357AETE_T

Commit message: main PCB v1 done
Parts:
- removed H201, H202, H203, H204: MountingHole, MountingHole:MountingHole_3.7mm, symbol Mechanical:MountingHole
- removed H205, H206: MountingHole, MountingHole:MountingHole_3.2mm_M3, symbol Mechanical:MountingHole
- removed MK201: ICS-43434, ICS_43434(MIC):MIC_ICS-43434, symbol ICS-43434:ICS-43434
- removed R202: 100k, Resistor_SMD:R_0805_2012Metric_Pad1.20x1.40mm_HandSolder, symbol Device:R
- added MK202: SPH0645LM4H-B, SPH0645LM4H-B(Microphone):MIC_SPH0645LM4H-B, symbol SPH0645LM4H-B:SPH0645LM4H-B
- added R204: 51, Resistor_SMD:R_0805_2012Metric_Pad1.20x1.40mm_HandSolder, symbol Device:R
- added R205: 100k, Resistor_SMD:R_0805_2012Metric_Pad1.20x1.40mm_HandSolder, symbol Device:R
Connections:
- net +3.3V: now also MK202.5 (VDD)
- net GND: now also MK202.2 (SELECT), MK202.3 (GND), R205.2
- net MIC_I2S3_SCK: now also MK202.4 (BCLK)
- net MIC_I2S3_SD: now also R204.1, R205.1
- net MIC_I2S3_WS: now also MK202.1 (WS)
- new net: MK202.6 (DATA_OUT), R204.2
Other:
- note added: "SELECT = LOW the DATA pin drives the SDIN bus when WS = LOW otherwise DATA = tri-state."
