File: Portable Offline Translator/MCU.kicad_sch (KiCad schematic)
At the start: 22 parts

Commit message: Added Datasheets and PCB
Parts:
- added R306, R307: 10k, Resistor_SMD:R_0805_2012Metric_Pad1.20x1.40mm_HandSolder, symbol Device:R
- added SW302, SW303: SW_Push, Button_Switch_SMD:SW_SPST_B3S-1000, symbol Switch:SW_Push
- C301, C302, C303, C304, C305, C306, C307, C308, C309, C310, C311: renamed from C?; footprint Capacitor_SMD:C_0603_1608Metric -> Capacitor_SMD:C_0603_1608Metric_Pad1.08x0.95mm_HandSolder
- R301, R303, R305: renamed from R?; footprint Resistor_SMD:R_0603_1608Metric -> Resistor_SMD:R_0805_2012Metric_Pad1.20x1.40mm_HandSolder
- R302, R304: renamed from R?; footprint Resistor_SMD:R_0402_1005Metric -> Resistor_SMD:R_0805_2012Metric_Pad1.20x1.40mm_HandSolder
- gave numbers to parts that had none: 6
Connections:
- net GND: now also R306.2, R307.2
- net NRST: now also U301.J1 (NRST)
- net at U301.A11 (PD7): now also SW303.1
- net at U301.C15 (PA11): now also SW302.1
- net LCD_Data/Command: now reaches U301.E15 (PA9)
- net LCD_RST: now reaches U301.F15 (PA8)
- new net +5V: R306.1, R307.1, SW302.2, SW303.2

Commit message: PCB Backup
Parts:
- added R308: 10k, Resistor_SMD:R_0805_2012Metric_Pad1.20x1.40mm_HandSolder, symbol Device:R
- added SW304: SW_Push, Button_Switch_SMD:SW_SPST_B3S-1000, symbol Switch:SW_Push
Connections:
- net +5V: now also R308.1, SW304.2
- net GND: now also R308.2
- net at U301.C10 (PG9): now also SW304.1
Changed lines of the file:
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@@
   (junction (at 44.45 52.07) (diameter 0) (color 0 0 0 0)
+  )
+  (junction (at 118.11 193.04) (diameter 0) (color 0 0 0 0)
   )
   (junction (at 214.63 261.62) (diameter 0) (color 0 0 0 0)
@@
     (stroke (width 0) (type default) (color 0 0 0 0))
   )
+  (wire (pts (xy 118.11 205.74) (xy 118.11 193.04))
+    (stroke (width 0) (type default) (color 0 0 0 0))
+  )
   (wire (pts (xy 196.85 261.62) (xy 196.85 259.08))
     (stroke (width 0) (type default) (color 0 0 0 0))
@@
     (stroke (width 0) (type default) (color 0 0 0 0))
   )
+  (wire (pts (xy 118.11 180.34) (xy 118.11 175.26))
+    (stroke (width 0) (type default) (color 0 0 0 0))
+  )
   (wire (pts (xy 237.49 259.08) (xy 237.49 261.62))
     (stroke (width 0) (type default) (color 0 0 0 0))
@@
     (stroke (width 0) (type default) (color 0 0 0 0))
   )
+  (wire (pts (xy 124.46 193.04) (xy 118.11 193.04))
+    (stroke (width 0) (type default) (color 0 0 0 0))
+  )
   (wire (pts (xy 73.66 146.05) (xy 73.66 137.16))
     (stroke (width 0) (type default) (color 0 0 0 0))
@@
     (stroke (width 0) (type default) (color 0 0 0 0))
   )
+  (wire (pts (xy 158.75 193.04) (xy 134.62 193.04))
+    (stroke (width 0) (type default) (color 0 0 0 0))
+  )
   (wire (pts (xy 181.61 261.62) (xy 182.88 261.62))
     (stroke (width 0) (type default) (color 0 0 0 0))
@@
   )
   (wire (pts (xy 102.87 60.96) (xy 102.87 62.23))
+    (stroke (width 0) (type default) (color 0 0 0 0))
+  )
+  (wire (pts (xy 118.11 193.04) (xy 118.11 187.96))
     (stroke (width 0) (type default) (color 0 0 0 0))
   )
@@
     (pin "2")
   )
+  (symbol (lib_id "Switch:SW_Push") (at 129.54 193.04 180) (unit 1)
+    (in_bom yes) (on_board yes) (fields_autoplaced)
+    (property "Reference" "SW304" (id 0) (at 129.54 200.66 0))
+    (property "Value" "SW_Push" (id 1) (at 129.54 198.12 0))
+    (property "Footprint" "Button_Switch_SMD:SW_SPST_B3S-1000" (id 2) (at 129.54 198.12 0)
+      (effects (font (size 1.27 1.27)) hide)
+    )
+    (property "Datasheet" "https://www.digikey.com/en/products/detail/omron-electronics-inc-emc-div/B3S-1000/20686" (id 3) (at 129.54 198.12 0)
+      (effects (font (size 1.27 1.27)) hide)
+    )
+    (pin "1")
+    (pin "2")
+  )
   (symbol (lib_id "power:+3V3") (at 102.87 49.53 0) (unit 1)
     (in_bom yes) (on_board yes) (fields_autoplaced)
@@
     (pin "1")
     (pin "2")
+  )
+  (symbol (lib_id "power:GND") (at 118.11 175.26 180) (unit 1)
+    (in_bom yes) (on_board yes) (fields_autoplaced)
+    (property "Reference" "#PWR0134" (id 0) (at 118.11 168.91 0)
+      (effects (font (size 1.27 1.27)) hide)
+    )
+    (property "Value" "GND" (id 1) (at 118.11 170.18 0))
+    (property "Footprint" "" (id 2) (at 118.11 175.26 0)
+      (effects (font (size 1.27 1.27)) hide)
+    )
+    (property "Datasheet" "" (id 3) (at 118.11 175.26 0)
+      (effects (font (size 1.27 1.27)) hide)
+    )
+    (pin "1")
   )
   (symbol (lib_id "power:GND") (at 182.88 264.16 0) (unit 1)
@@
     (pin "2")
   )
+  (symbol (lib_id "Device:R") (at 118.11 184.15 180) (unit 1)
+    (in_bom yes) (on_board yes) (fields_autoplaced)
+    (property "Reference" "R308" (id 0) (at 115.57 185.4201 0)
+      (effects (font (size 1.27 1.27)) (justify left))
+    )
+    (property "Value" "10k" (id 1) (at 115.57 182.8801 0)
+      (effects (font (size 1.27 1.27)) (justify left))
+    )
+    (property "Footprint" "Resistor_SMD:R_0805_2012Metric_Pad1.20x1.40mm_HandSolder" (id 2) (at 119.888 184.15 90)
+      (effects (font (size 1.27 1.27)) hide)
+    )
+    (property "Datasheet" "~" (id 3) (at 118.11 184.15 0)
+      (effects (font (size 1.27 1.27)) hide)
+    )
+    (pin "1")
+    (pin "2")
+  )
   (symbol (lib_id "power:+3V3") (at 40.64 45.72 0) (unit 1)
     (in_bom yes) (on_board yes) (fields_autoplaced)
@@
     (pin "2")
   )
+  (symbol (lib_id "power:+5V") (at 118.11 205.74 180) (unit 1)
+    (in_bom yes) (on_board yes) (fields_autoplaced)
+    (property "Reference" "#PWR0133" (id 0) (at 118.11 201.93 0)
+      (effects (font (size 1.27 1.27)) hide)
+    )
+    (property "Value" "+5V" (id 1) (at 118.11 210.82 0))
+    (property "Footprint" "" (id 2) (at 118.11 205.74 0)
+      (effects (font (size 1.27 1.27)) hide)
+    )
+    (property "Datasheet" "" (id 3) (at 118.11 205.74 0)
+      (effects (font (size 1.27 1.27)) hide)
+    )
+    (pin "1")
+  )
   (symbol (lib_id "Connector:TestPoint") (at 176.53 261.62 90) (unit 1)

Commit message: PCB iteration 1
Parts:
- removed C310: 10n, Capacitor_SMD:C_0603_1608Metric_Pad1.08x0.95mm_HandSolder, symbol basic:C
- removed C311: 1u, Capacitor_SMD:C_0603_1608Metric_Pad1.08x0.95mm_HandSolder, symbol basic:C
- removed R302, R304: 2k2, Resistor_SMD:R_0805_2012Metric_Pad1.20x1.40mm_HandSolder, symbol Device:R_Small
- removed R306, R308: 10k, Resistor_SMD:R_0805_2012Metric_Pad1.20x1.40mm_HandSolder, symbol Device:R
- removed SW302, SW304: SW_Push, Button_Switch_SMD:SW_SPST_B3S-1000, symbol Switch:SW_Push
- removed TP302: GND, TestPoint:TestPoint_Keystone_5000-5004_Miniature, symbol Connector:TestPoint
- removed U301: STM32F407IEHx, Package_BGA:UFBGA-201_10x10mm_Layout15x15_P0.65mm, symbol MCU_ST_STM32F4:STM32F407IEHx
- added IC301: STM32F407IET6, Package_QFP:LQFP-176_24x24mm_P0.5mm, symbol STM32F407IET6:STM32F407IET6
- added R309, R310: 10k, Resistor_SMD:R_0805_2012Metric_Pad1.20x1.40mm_HandSolder, symbol Device:R
- added SW305, SW306: SW_Push, Button_Switch_SMD:SW_SPST_B3S-1000, symbol Switch:SW_Push
Connections:
- net +5V: now also R309.1, R310.1, SW305.2, SW306.2
- net BOOT0: now also IC301.166 (BOOT0)
- net BOOT1: now also J301.4 (Pin_4), R303.1, IC301.58 (PB2)
- net GND: now also IC301.102 (VSS_6), IC301.113 (VSS_7), IC301.126 (VSS_8), IC301.135 (VSS_9), IC301.14 (VSS_1), IC301.148 (VSS_10), IC301.158 (VSS_11), IC301.61 (VSS_3), IC301.71 (VSS_4), IC301.90 (VSS_5), R309.2, R310.2
- net I2S2_CK: now also IC301.93 (PB13)
- net I2S2_SD: now also IC301.95 (PB15)
- net I2S2_WS: now also IC301.92 (PB12)
- net I2S3_CK: now also IC301.139 (PC10)
- net I2S3_SD: now also IC301.141 (PC12)
- net I2S3_WS: now also IC301.138 (PA15)
- net LCD_Data/Command: now also IC301.120 (PA9)
- net LCD_RST: now also IC301.119 (PA8)
- net NRST: now also IC301.31 (NRST)
- net OSC_IN: now also IC301.29 (PH0)
- net OSC_OUT: now also IC301.30 (PH1)
- net SPI1_MOSI: now also IC301.53 (PA7)
- net SPI1_NSS: now also IC301.50 (PA4)
- net SPI1_SCK: now also IC301.51 (PA5)
- net SPI_MISO: now also IC301.52 (PA6)
- net at SW303.1: now also IC301.151 (PD7)
- net +3V3 renamed +3.3V
- net +3.3V: now also IC301.103 (VDD_9), IC301.114 (VDD_10), IC301.127 (VDD_11), IC301.136 (VDD_12), IC301.149 (VDD_13), IC301.15 (VDD_1), IC301.159 (VDD_14), IC301.172 (VDD_15), IC301.49 (VDD_4), IC301.62 (VDD_5), IC301.72 (VDD_6), IC301.82 (VDD_7), IC301.91 (VDD_8)
- new net: IC301.122 (PA11), SW306.1
- new net: IC301.152 (PG9), SW305.1
- new net SPI2_MISO: IC301.34 (PC2)
- new net SPI2_MOSI: IC301.35 (PC3)
- new net SPI2_NSS: IC301.131 (PI0)
- new net SPI2_SCLK: IC301.79 (PB10)
- no-connect marks 1 -> 132
Other:
- note added: "I2S2 = AMP+SPKER I2S3 = MIC SPI = LCD SPI2 = RPI CM5"
- note removed: "I2S2 = AMP+SPKER I2S3 = MIC SPI = LCD I2C1 = RPI CM5"
- moved on the sheet: R307, SW303

Commit message: main PCB v1 done
Parts:
- added J3: Conn_ARM_JTAG_SWD_10, Connector_IDC:IDC-Header_2x05_P2.54mm_Vertical, symbol Connector:Conn_ARM_JTAG_SWD_10
- added R2, R5, R6: 100k, Resistor_SMD:R_0805_2012Metric_Pad1.20x1.40mm_HandSolder, symbol basic:R
Connections:
- net +3.3V: now also J3.1 (VTref), R2.1, R5.1, R6.1
- net GND: now also J3.3 (GND), J3.5 (GND), J3.9 (GNDDetect)
- net NRST: now also J3.10 (~{RESET})
- net JTMS/SWDIO: now reaches IC301.124 (PA13)
- net JTMS/SWDIO: now also J3.2 (SWDIO/TMS), R5.2
- net JTCK/SWCLK: now reaches IC301.129 (PH14)
- net JTCK/SWCLK: now also J3.4 (SWDCLK/TCK), R2.2
- net JTDO/TRACESWO: now reaches IC301.161 (PB3)
- net JTDO/TRACESWO: now also J3.6 (SWO/TDO), R6.2
- no-connect marks 132 -> 130
Other:
- note added: "Debug Header"
