File: Portable Offline Translator/Portable Offline Translator.kicad_pcb (KiCad board)
At the start: 2 copper layers, 49 parts, among them J201 Conn_01x10_Female, J301 Conn_02x03_Odd_Even, SW301 SW_Push, SW302 SW_Push, SW303 SW_Push, U201 MAX98357AEWL+T, U301 STM32F407IEHx, U401 LM317_SOT-223, U402 LM317_SOT-223, Y301 Crystal

Commit message: PCB Backup
Parts:
- added R308: 10k, Resistor_SMD:R_0805_2012Metric_Pad1.20x1.40mm_HandSolder, F.Cu at (182.0, 136.8)
- added SW304: SW_Push, Button_Switch_SMD:SW_SPST_B3S-1000, F.Cu at (182.1, 145.5)
- J201: value Conn_01x10_Female -> Conn_01x08_Male; footprint Connector_PinSocket_2.54mm:PinSocket_1x10_P2.54mm_Vertical -> Connector_PinSocket_2.54mm:PinSocket_1x08_P2.54mm_Vertical
- moved MK201 19.0 mm to (109.6, 126.9)
- moved LS201 15.0 mm to (93.9, 101.5)
- turned C404 to -90 degrees
Connections:
- J201 pad 1: /IO Circuits/I2C1_SCL -> /IO Circuits/LCD_VCC
- J201 pad 2: /IO Circuits/I2C1_SDA -> GND
- J201 pad 3: /IO Circuits/LCD_Data/Command -> /IO Circuits/SPI_MISO
- J201 pad 4: /IO Circuits/LCD_RST -> /IO Circuits/SPI1_SCK
- J201 pad 5: /IO Circuits/SPI1_NSS -> /IO Circuits/SPI1_MOSI
- J201 pad 6: /IO Circuits/SPI1_MOSI -> /IO Circuits/SPI1_NSS
- J201 pad 7: /IO Circuits/SPI_MISO -> /IO Circuits/LCD_Data/Command
- J201 pad 8: /IO Circuits/SPI1_SCK -> /IO Circuits/LCD_RST
- R302 pad 2: /IO Circuits/I2C1_SCL -> /MCU/I2C1_SCL
- R304 pad 2: /IO Circuits/I2C1_SDA -> /MCU/I2C1_SDA
- U301 pad B5: /IO Circuits/I2C1_SDA -> /MCU/I2C1_SDA
- U301 pad B6: /IO Circuits/I2C1_SCL -> /MCU/I2C1_SCL
- U301 pad C10: unconnected-(U301-PadC10) -> Net-(SW304-Pad1)
Routing:
- net +3.3V: track 0.00 -> 58.6 mm, vias 0 -> 2
- net Net-(C404-Pad1): track 0.00 -> 35.6 mm
- net /PowerSS/REG_IN: track 101.5 -> 110.0 mm
- net Net-(C403-Pad1): track 26.8 -> 35.2 mm
- net +5V: track 39.7 -> 46.8 mm, vias 0 -> 1

Commit message: PCB iteration 1
Parts:
- removed R201: 100k, Resistor_SMD:R_0805_2012Metric_Pad1.20x1.40mm_HandSolder
- removed R302, R304: 2k2, Resistor_SMD:R_0805_2012Metric_Pad1.20x1.40mm_HandSolder
- removed R306: 10k, Resistor_SMD:R_0805_2012Metric_Pad1.20x1.40mm_HandSolder
- removed SW302, SW304: SW_Push, Button_Switch_SMD:SW_SPST_B3S-1000
- removed U201: MAX98357AEWL+T, MAX98357AEWL_T(Audio Amp):21-0896B_9_MXM
- removed U301: STM32F407IEHx, Package_BGA:UFBGA-201_10x10mm_Layout15x15_P0.65mm
- added H201: MountingHole, MountingHole:MountingHole_3.7mm, F.Cu at (85.2, 99.5)
- added H202: MountingHole, MountingHole:MountingHole_3.7mm, F.Cu at (118.4, 99.6)
- added H203: MountingHole, MountingHole:MountingHole_3.7mm, F.Cu at (85.4, 147.6)
- added H204: MountingHole, MountingHole:MountingHole_3.7mm, F.Cu at (118.5, 147.6)
- added H205: MountingHole, MountingHole:MountingHole_3.2mm_M3, F.Cu at (108.5, 39.6)
- added H206: MountingHole, MountingHole:MountingHole_3.2mm_M3, F.Cu at (163.8, 39.8)
- added IC301: STM32F407IET6, Package_QFP:LQFP-176_24x24mm_P0.5mm, F.Cu at (153.3, 107.2)
- added Module201: ComputeModule5-CM5, CM5IO:Raspberry-Pi-5-Compute-Module, F.Cu at (85.4, 147.6)
- added R203: 100k, Resistor_SMD:R_0805_2012Metric_Pad1.20x1.40mm_HandSolder, F.Cu at (180.6, 119.5)
- added R309: 10k, Resistor_SMD:R_0805_2012Metric_Pad1.20x1.40mm_HandSolder, F.Cu at (150.5, 141.7)
- added R310: 10k, Resistor_SMD:R_0805_2012Metric_Pad1.20x1.40mm_HandSolder, F.Cu at (165.5, 141.0)
- added SW305: SW_Push, Button_Switch_SMD:SW_SPST_B3S-1000, F.Cu at (151.5, 133.7)
- added SW306: SW_Push, Button_Switch_SMD:SW_SPST_B3S-1000, F.Cu at (165.6, 133.2)
- added TP303: SPI4_CSn, TestPoint:TestPoint_Keystone_5000-5004_Miniature, F.Cu at (88.1, 91.1)
- added TP304: SPI4_MOSI, TestPoint:TestPoint_Keystone_5000-5004_Miniature, F.Cu at (93.1, 90.9)
- added TP305: SPI4_MISO, TestPoint:TestPoint_Keystone_5000-5004_Miniature, F.Cu at (99.1, 90.9)
- added TP306: SPI4_SCLK, TestPoint:TestPoint_Keystone_5000-5004_Miniature, F.Cu at (82.9, 90.9)
- added TP308: I2S_CLK, TestPoint:TestPoint_Keystone_5000-5004_Miniature, F.Cu at (174.0, 126.5)
- added TP309: 3.3V, TestPoint:TestPoint_Keystone_5000-5004_Miniature, F.Cu at (183.5, 128.4)
- added U202: MAX98357AETE_T, Package_DFN_QFN:TQFN-16-1EP_3x3mm_P0.5mm_EP1.23x1.23mm, F.Cu at (175.7, 119.1)
- TP302: value GND -> 5V
- moved TP302 40.1 mm to (185.8, 139.7)
- moved J201 30.4 mm to (157.4, 150.5)
- moved LS201 22.0 mm to (112.9, 90.4), turned to 90 degrees
- moved MK201 20.4 mm to (129.6, 122.8)
- moved C305 19.0 mm to (187.8, 131.2)
- moved C303 19.0 mm to (187.7, 120.8)
- moved C304 19.0 mm to (187.7, 126.0)
- moved C307 19.0 mm to (194.7, 125.6)
- moved C308 19.0 mm to (194.5, 120.7)
- moved C309 19.0 mm to (194.4, 131.2)
- moved C311 18.9 mm to (194.8, 113.3)
- moved TP301 18.9 mm to (180.2, 111.6)
- moved C310 18.9 mm to (187.7, 113.4)
- moved R202 18.0 mm to (128.6, 88.2)
- moved R307 17.6 mm to (137.4, 141.1)
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Connections:
- net OSC_IN renamed /MCU/OSC_IN
- net OSC_OUT renamed /MCU/OSC_OUT
- C303 pad 1: +3V3 -> +3.3V
- C304 pad 1: +3V3 -> +3.3V
- C305 pad 1: +3V3 -> +3.3V
- C307 pad 1: +3V3 -> +3.3V
- C308 pad 1: +3V3 -> +3.3V
- C309 pad 1: +3V3 -> +3.3V
- C310 pad 1: +3V3 -> +3.3V
- C311 pad 1: +3V3 -> +3.3V
- J201 pad 1: /IO Circuits/LCD_VCC -> +3.3V
- J201 pad 3: /IO Circuits/SPI_MISO -> /IO Circuits/SPI1_MOSI
- J201 pad 4: /IO Circuits/SPI1_SCK -> /IO Circuits/SPI_MISO
- J201 pad 5: /IO Circuits/SPI1_MOSI -> /IO Circuits/SPI1_SCK
- J301 pad 1: +3V3 -> +3.3V
- J301 pad 2: +3V3 -> +3.3V
- J301 pad 4: Net-(J301-Pad4) -> BOOT1
- R303 pad 1: Net-(J301-Pad4) -> BOOT1
- R305 pad 1: +3V3 -> +3.3V
- TP301 pad 1: +3V3 -> +3.3V
- TP302 pad 1: GND -> +5V
Routing:
- net +3.3V: track 58.6 -> 461.0 mm, vias 2 -> 17
- net +5V: track 46.8 -> 300.0 mm, vias 1 -> 7
- net GND: track 0.00 -> 221.1 mm, vias 2 -> 23
- net /IO Circuits/SPI4_CSn: track 0.00 -> 144.3 mm, vias 0 -> 2
- net /IO Circuits/SPI4_SCLK: track 0.00 -> 127.5 mm, vias 0 -> 4
- net /IO Circuits/LCD_RST: track 0.00 -> 125.5 mm, vias 0 -> 4
- net /MCU/NRST: track 0.00 -> 119.0 mm, vias 0 -> 2
- net /IO Circuits/LCD_Data/Command: track 0.00 -> 115.2 mm, vias 0 -> 2
- net /IO Circuits/SPI4_MISO: track 0.00 -> 112.8 mm, vias 0 -> 2
- net /IO Circuits/SPI4_MOSI: track 0.00 -> 112.4 mm, vias 0 -> 2
- net BOOT1: track 0.00 -> 92.5 mm, vias 0 -> 4
- net Net-(IC301-PG9): track 0.00 -> 82.0 mm, vias 0 -> 4
- net /IO Circuits/OUTP: track 0.00 -> 81.7 mm, vias 0 -> 2
- net /IO Circuits/OUTN: track 0.00 -> 81.0 mm, vias 0 -> 2
- net Net-(IC301-PD7): track 0.00 -> 78.9 mm, vias 0 -> 4
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Other:
- board outline added: 121.4 x 144.4 mm
- board text added: "3.3V"
- board text added: "AMP_CLK"
- board text added: "AMP_WS"
- board text added: "CM5_CSn"
- board text added: "CM5_MISO"
- board text added: "CM5_MOSI"
- board text added: "CM5_SCLK"
- board text added: "DEST LANG"
- board text added: "NRST"
- board text added: "SRC LANG"
- board text added: "START"

Commit message: PCB iteration1 gerber and drill files added
Parts:
- removed H201, H202, H203, H204: MountingHole, MountingHole:MountingHole_3.7mm

Commit message: main PCB v1 done
Parts:
- removed BT401: 1048P, 1048P(16850 Dual Bat Holder:BAT_1048P
- removed H205, H206: MountingHole, MountingHole:MountingHole_3.2mm_M3
- removed MK201: ICS-43434, ICS_43434(MIC):MIC_ICS-43434
- added J3: Conn_ARM_JTAG_SWD_10, Connector_IDC:IDC-Header_2x05_P2.54mm_Vertical, F.Cu at (84.3, 61.8)
- added J401: B2B-XH-A, Battery Connector(JST-XH):JST_B2B-XH-A, F.Cu at (118.4, 58.9)
- added MK202: SPH0645LM4H-B, SPH0645LM4H-B(Microphone):MIC_SPH0645LM4H-B, F.Cu at (129.5, 123.6)
- added R2: 100k, Resistor_SMD:R_0805_2012Metric_Pad1.20x1.40mm_HandSolder, F.Cu at (166.3, 79.2)
- added R204: 51, Resistor_SMD:R_0805_2012Metric_Pad1.20x1.40mm_HandSolder, F.Cu at (117.3, 108.3)
- added R205: 100k, Resistor_SMD:R_0805_2012Metric_Pad1.20x1.40mm_HandSolder, F.Cu at (117.3, 105.3)
- added R5: 100k, Resistor_SMD:R_0805_2012Metric_Pad1.20x1.40mm_HandSolder, F.Cu at (163.3, 80.3)
- added R6: 100k, Resistor_SMD:R_0805_2012Metric_Pad1.20x1.40mm_HandSolder, F.Cu at (160.3, 80.3)
- moved R308 117.8 mm to (84.8, 70.2)
- moved TP302 117.8 mm to (88.6, 73.2)
- moved C309 78.8 mm to (157.5, 61.6)
- moved C305 72.6 mm to (157.5, 65.2)
- moved C308 67.2 mm to (152.4, 68.3)
- moved C311 64.6 mm to (152.4, 64.6)
- moved C307 64.4 mm to (152.8, 76.8)
- moved C310 62.9 mm to (152.1, 61.6)
- moved TP301 62.8 mm to (141.4, 62.4)
- moved C304 62.3 mm to (152.9, 74.3)
- moved C303 60.7 mm to (152.6, 71.2)
- moved C306 53.4 mm to (128.0, 140.6)
- moved SW301 49.6 mm to (128.3, 146.7)
- moved R305 49.0 mm to (137.8, 146.7)
- moved R203 25.1 mm to (174.6, 95.1)
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Connections:
- IC301 pad 124: unconnected-(IC301-PA13-Pad124) -> /MCU/JTMS/SWDIO
- IC301 pad 129: unconnected-(IC301-PH14-Pad129) -> /MCU/JTCK/SWCLK
- IC301 pad 161: unconnected-(IC301-PB3-Pad161) -> /MCU/JTDO/TRACESWO
Routing:
- net /MCU/JTMS/SWDIO: track 0.00 -> 137.1 mm, vias 0 -> 3
- net /MCU/JTCK/SWCLK: track 0.00 -> 131.5 mm, vias 0 -> 2
- net /MCU/JTDO/TRACESWO: track 0.00 -> 111.9 mm, vias 0 -> 1
- net /PowerSS/REG_IN: track 134.5 -> 91.6 mm
- net /MCU/NRST: track 119.0 -> 160.0 mm, vias 2 -> 5
- net +3.3V: track 461.0 -> 497.7 mm
- net /IO Circuits/LCD_RST: track 125.5 -> 95.3 mm, vias 4 -> 2
- net /IO Circuits/LCD_Data/Command: track 115.2 -> 92.0 mm, vias 2 -> 4
- net Net-(MK202-DATA_OUT): track 0.00 -> 21.0 mm, vias 0 -> 2
- net +5V: track 300.0 -> 320.7 mm
- net Net-(BT401-PadN1): track 19.1 -> 0.00 mm
- net /IO Circuits/AMP_I2S2_SD: track 31.1 -> 12.3 mm
- net Net-(U202-GAIN_SLOT): track 2.53 -> 19.3 mm
- net Net-(IC301-PA11): track 65.8 -> 50.5 mm
- net /IO Circuits/OUTN: track 81.0 -> 90.1 mm, vias 2 -> 4
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Other:
- board size 121.4 x 144.4 mm -> 99.7 x 99.8 mm
