File: Portable Offline Translator/Portable Offline Translator.kicad_sch (KiCad schematic)
At the start: 41 parts

Commit message: MCU and Power SS updated
Parts:
- removed BT?: Battery_Cell, Battery:BatteryHolder_Keystone_3000_1x12mm, symbol Device:Battery_Cell
- removed C?: 4.7u, Capacitor_SMD:C_0603_1608Metric, symbol basic:C
- removed C? (x2): 14p, Capacitor_SMD:C_0402_1005Metric, symbol basic:C
- removed C?: 1u, Capacitor_SMD:C_0603_1608Metric, symbol basic:C
- removed C?: 10n, Capacitor_SMD:C_0603_1608Metric, symbol basic:C
- removed C? (x5): 100n, Capacitor_SMD:C_0603_1608Metric, symbol basic:C
- removed TP?: GND, TestPoint:TestPoint_Keystone_5000-5004_Miniature, symbol Connector:TestPoint
- removed TP?: 3V3, TestPoint:TestPoint_Keystone_5000-5004_Miniature, symbol Connector:TestPoint
- removed U?: STM32F103C8Tx, Package_QFP:LQFP-48_7x7mm_P0.5mm, symbol MCU_ST_STM32F1:STM32F103C8Tx
- removed Y?: Crystal, Crystal:Crystal_SMD_3215-2Pin_3.2x1.5mm, symbol Device:Crystal
- added C?: 10n, Capacitor_SMD:C_0603_1608Metric, symbol basic:C
- added C? (x5): 100n, Capacitor_SMD:C_0603_1608Metric, symbol basic:C
- added C?: 1u, Capacitor_SMD:C_0603_1608Metric, symbol basic:C
- added C?: 4.7u, Capacitor_SMD:C_0603_1608Metric, symbol basic:C
- added R? (x2): 2k2, Resistor_SMD:R_0402_1005Metric, symbol Device:R_Small
- added TP?: GND, TestPoint:TestPoint_Keystone_5000-5004_Miniature, symbol Connector:TestPoint
- added TP?: 3.3V, TestPoint:TestPoint_Keystone_5000-5004_Miniature, symbol Connector:TestPoint
- added U?: STM32F407IEHx, Package_BGA:UFBGA-201_10x10mm_Layout15x15_P0.65mm, symbol MCU_ST_STM32F4:STM32F407IEHx
Connections:
- net +3V3: now also C?.1, C?.1, C?.1, C?.1, C?.1, C?.1, C?.1, C?.1, R?.1, R?.1, TP?.1, U?.C1 (VBAT), U?.C5 (VDD), U?.C7 (VDD), U?.C8 (VDD), U?.C9 (VDD), U?.F3 (VDD), U?.G13 (VDD), U?.G3 (VDD), U?.H13 (VDD), U?.J12 (VDD), U?.J13 (VDD), U?.K4 (VDD), U?.N10 (VDD), U?.N8 (VDD), U?.N9 (VDD), U?.R1 (VDDA)
- net BOOT0: now also U?.D6 (BOOT0)
- net BOOT1: now also U?.M6 (PB2); no longer J?.4 (Pin_4), R?.1
- net GND: now also BT?.N2, C?.2, C?.2, C?.2, C?.2, C?.2, C?.2, C?.2, C?.2, TP?.1, U?.D5 (VSS), U?.D7 (VSS), U?.D8 (VSS), U?.D9 (VSS), U?.F10 (VSS), U?.F12 (VSS), U?.F2 (VSS), U?.F6 (VSS), U?.F7 (VSS), U?.F8 (VSS), U?.F9 (VSS), U?.G10 (VSS), U?.G12 (VSS), U?.G2 (VSS), U?.G6 (VSS), U?.G7 (VSS), U?.G8 (VSS), U?.G9 (VSS), U?.H10 (VSS), U?.H12 (VSS), U?.H6 (VSS), U?.H7 (VSS), U?.H8 (VSS), U?.H9 (VSS), U?.J10 (VSS), U?.J6 (VSS), U?.J7 (VSS), U?.J8 (VSS), U?.J9 (VSS), U?.K10 (VSS), U?.K6 (VSS), U?.K7 (VSS), U?.K8 (VSS), U?.K9 (VSS), U?.M1 (VSSA), U?.M8 (VSS), U?.M9 (VSS)
- net OSC_IN: now also U?.G1 (PH0)
- net OSC_OUT: now also U?.H1 (PH1)
- net REG_IN: now also BT?.P1
- net SPI1_MOSI: now also U?.R3 (PA7)
- net SPI1_NSS: now also U?.N4 (PA4)
- net SPI1_SCK: now also U?.P4 (PA5)
- net at BT?.N1: now also BT?.P2
- new net: J?.4 (Pin_4), R?.1
- new net I2C1_SCL: R?.2, U?.B6 (PB6)
- new net I2C1_SDA: R?.2, U?.B5 (PB7)
- new net SPI_MISO: U?.P3 (PA6)
- no-connect marks 0 -> 1
Other:
- moved on the sheet: BT?, C?, J?, R?, SW?, Y?

Commit message: IO schematic in prog
Parts:
- removed BT?: 1048P, 1048P:BAT_1048P, symbol 1048P:1048P
- removed C?: 10n, Capacitor_SMD:C_0603_1608Metric, symbol basic:C
- removed C? (x2): 10u, Capacitor_SMD:C_0603_1608Metric, symbol basic:C
- removed C? (x2): 20p, Capacitor_SMD:C_0603_1608Metric, symbol basic:C
- removed C? (x5): 100n, Capacitor_SMD:C_0603_1608Metric, symbol basic:C
- removed C? (x2): 1uF, symbol Device:C_Polarized_US
- removed C? (x2): 1u, Capacitor_SMD:C_0603_1608Metric, symbol basic:C
- removed C? (x2): 0.1uF, symbol Device:C_Polarized_US
- removed C?: 4.7u, Capacitor_SMD:C_0603_1608Metric, symbol basic:C
- removed D? (x4): 1N4002, Diode_THT:D_DO-41_SOD81_P10.16mm_Horizontal, symbol Diode:1N4002
- removed J?: Conn_02x03_Odd_Even, Connector_PinSocket_2.54mm:PinSocket_2x03_P2.54mm_Vertical, symbol Connector_Generic:Conn_02x03_Odd_Even
- removed R? (x2): 330, symbol Device:R
- removed R? (x3): 10k, Resistor_SMD:R_0603_1608Metric, symbol basic:R
- removed R? (x2): 2k2, Resistor_SMD:R_0402_1005Metric, symbol Device:R_Small
- removed R?: 1k, symbol Device:R
- removed R?: 542, symbol Device:R
- removed SW?: SW_Push, Button_Switch_SMD:SW_SPST_B3S-1000, symbol Switch:SW_Push
- removed TP?: GND, TestPoint:TestPoint_Keystone_5000-5004_Miniature, symbol Connector:TestPoint
- removed TP?: 3.3V, TestPoint:TestPoint_Keystone_5000-5004_Miniature, symbol Connector:TestPoint
- removed U?: STM32F407IEHx, Package_BGA:UFBGA-201_10x10mm_Layout15x15_P0.65mm, symbol MCU_ST_STM32F4:STM32F407IEHx
- removed U? (x2): LM317_SOT-223, Package_TO_SOT_SMD:SOT-223-3_TabPin2, symbol Regulator_Linear:LM317_SOT-223
- removed Y?: Crystal, Crystal:Crystal_HC49-U_Vertical, symbol Device:Crystal
Connections:
- no-connect marks 1 -> 0
Other:
- added sheet IO Circuits (IO.kicad_sch)
- added sheet MCU (MCU.kicad_sch)
- added sheet PowerSS (powerSS.kicad_sch)
- note added: "MCU->AMP+SPEAKER"
- note added: "MIC->MCU"
- note added: "TOP SHEET"
- note removed: "Connect 4.7u cap to V_dd3 (pin 48)"
- note removed: "Microcontroller"
- note removed: "Power Subsystem"

Commit message: Added Datasheets and PCB
Other:
- sheet IO Circuits ports: added I2C1_SCL, I2C1_SDA, LCD_Data/Command, LCD_GND, LCD_RST, LCD_VIN, SPI1_MOSI, SPI1_NSS, SPI1_SCK, SPI_MISO; removed none
- sheet MCU ports: added LCD_Data/Command, LCD_RST; removed none
- sheet PowerSS ports: added none; removed REG_IN
- note added: "MCU->LCD"
- note added: "MCU<->CM5"

Commit message: PCB iteration 1
Parts:
- added TP303: SPI4_CSn, TestPoint:TestPoint_Keystone_5000-5004_Miniature, symbol Connector:TestPoint
- added TP304: SPI4_MOSI, TestPoint:TestPoint_Keystone_5000-5004_Miniature, symbol Connector:TestPoint
- added TP305: SPI4_MISO, TestPoint:TestPoint_Keystone_5000-5004_Miniature, symbol Connector:TestPoint
- added TP306: SPI4_SCLK, TestPoint:TestPoint_Keystone_5000-5004_Miniature, symbol Connector:TestPoint
- added TP308: I2S_CLK, TestPoint:TestPoint_Keystone_5000-5004_Miniature, symbol Connector:TestPoint
- added TP309: 3.3V, TestPoint:TestPoint_Keystone_5000-5004_Miniature, symbol Connector:TestPoint
Connections:
- net IO Circuits/AMP_I2S2_CK: now also TP309.1
- net IO Circuits/AMP_I2S2_WS: now also TP308.1
- new net IO Circuits/SPI4_CSn: TP303.1
- new net IO Circuits/SPI4_MISO: TP305.1
- new net IO Circuits/SPI4_MOSI: TP304.1
- new net IO Circuits/SPI4_SCLK: TP306.1
Other:
- sheet IO Circuits ports: added LCD_VCC, SPI4_CSn, SPI4_MISO, SPI4_MOSI, SPI4_SCLK; removed I2C1_SCL, I2C1_SDA, LCD_VIN
- sheet MCU ports: added SPI2_MISO, SPI2_MOSI, SPI2_NSS, SPI2_SCLK; removed I2C1_SCL, I2C1_SDA
- note added: "AMP+SPEAKER -> MCU"
- note added: "CM5 <-> MCU"
- note added: "LCD <-> MCU"
- note added: "MIC -> MCU"
- note removed: "MCU->AMP+SPEAKER"
- note removed: "MCU->LCD"
- note removed: "MCU<->CM5"
- note removed: "MIC->MCU"
